File: vag-kcan-comm/vag-kcan-comm.kicad_sch (KiCad schematic)
At the start: 23 parts, among them J1 OBD2, J2 USB_A, Q1 2N7002, U1 TJA1042T, U2 LM339, U3 PIC18F25K80_ISS, U4 74AHCT125, U5 FT232RL, Y1 Crystal

Commit message: MCU reset on DTR line
Connections:
- net at U3.1 (~{MCLR}/RE3): now also U5.2 (DTR)
Changed lines of the file:
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@@
+	(wire
+		(pts
+			(xy 213.36 53.34) (xy 213.36 66.04)
+		)
+		(stroke
+			(width 0)
+			(type default)
+		)
+	)
 	(wire
 		(pts
@@
 	(wire
 		(pts
+			(xy 87.63 118.11) (xy 121.92 118.11)
+		)
+		(stroke
+			(width 0)
+			(type default)
+		)
+	)
+	(wire
+		(pts
 			(xy 203.2 66.04) (xy 209.55 66.04)
 		)
@@
 	(wire
 		(pts
+			(xy 121.92 53.34) (xy 213.36 53.34)
+		)
+		(stroke
+			(width 0)
+			(type default)
+		)
+	)
+	(wire
+		(pts
 			(xy 139.7 123.19) (xy 226.06 123.19)
 		)
@@
 	(wire
 		(pts
+			(xy 121.92 118.11) (xy 121.92 53.34)
+		)
+		(stroke
+			(width 0)
+			(type default)
+		)
+	)
+	(wire
+		(pts
 			(xy 226.06 123.19) (xy 226.06 146.05)
 		)
@@
 		)
 		(stroke
+			(width 0)
+			(type default)
+		)
+	)
+	(wire
+		(pts
+			(xy 213.36 66.04) (xy 218.44 66.04)
+		)
+		(stroke
